Commit message: Configure TurtleBot3 differential drive control

File: src/turtlebot3_mujoco_sim/description/turtlebot3_burger.urdf.xacro (robot description, xacro)
@@ -10,4 +10,18 @@
   -->
   <link name="base_link"/>
+  <link name="wheel_left_link"/>
+  <joint name="wheel_left" type="continuous">
+    <parent link="base_link"/>
+    <child link="wheel_left_link"/>
+    <origin xyz="0 0.08 0.033" rpy="-1.5708 0 0"/>
+    <axis xyz="0 0 1"/>
+  </joint>
+  <link name="wheel_right_link"/>
+  <joint name="wheel_right" type="continuous">
+    <parent link="base_link"/>
+    <child link="wheel_right_link"/>
+    <origin xyz="0 -0.08 0.033" rpy="-1.5708 0 0"/>
+    <axis xyz="0 0 1"/>
+  </joint>
   <ros2_control name="MujocoSystem" type="system">
     <hardware>
