Commit message: Add ROS 2 control launch and configurable UR5e initial pose

File: src/ur5e_mujoco_sim/generated/ur5e.urdf (robot description, URDF)
Before this commit: robot ur5e, 13 links, 12 joints
Links:
- link base_link_inertia: geometry collision mesh filename=file:///home/sohaib/MuJoCoROSTrippleS/install/ur_descriptio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; visual mesh filename=file:///home/sohaib/MuJoCoROSTrippleS/install/ur_descriptio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
- link forearm_link: geometry collision mesh filename=file:///home/sohaib/MuJoCoROSTrippleS/install/ur_descriptio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; visual mesh filename=file:///home/sohaib/MuJoCoROSTrippleS/install/ur_descriptio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
- link shoulder_link: geometry collision mesh filename=file:///home/sohaib/MuJoCoROSTrippleS/install/ur_descriptio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; visual mesh filename=file:///home/sohaib/MuJoCoROSTrippleS/install/ur_descriptio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
- link upper_arm_link: geometry collision mesh filename=file:///home/sohaib/MuJoCoROSTrippleS/install/ur_descriptio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; visual mesh filename=file:///home/sohaib/MuJoCoROSTrippleS/install/ur_descriptio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
- link wrist_1_link: geometry collision mesh filename=file:///home/sohaib/MuJoCoROSTrippleS/install/ur_descriptio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; visual mesh filename=file:///home/sohaib/MuJoCoROSTrippleS/install/ur_descriptio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
- link wrist_2_link: geometry collision mesh filename=file:///home/sohaib/MuJoCoROSTrippleS/install/ur_descriptio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; visual mesh filename=file:///home/sohaib/MuJoCoROSTrippleS/install/ur_descriptio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
- link wrist_3_link: geometry collision mesh filename=file:///home/sohaib/MuJoCoROSTrippleS/install/ur_descriptio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; visual mesh filename=file:///home/sohaib/MuJoCoROSTrippleS/install/ur_descriptio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

File: src/ur5e_mujoco_sim/urdf/ur5e.urdf.xacro (robot description, xacro)
@@ -3,4 +3,13 @@
   xmlns:xacro="http://www.ros.org/wiki/xacro"
   name="ur5e">
+  <xacro:arg
+    name="mujoco_model"
+    default="$(find ur5e_mujoco_sim)/generated/mjcf/mujoco_description_formatted.xml"/>
+  <xacro:arg
+    name="initial_positions_file"
+    default="$(find ur5e_mujoco_sim)/config/initial_positions.yaml"/>
+  <xacro:property
+    name="initial_positions"
+    value="${xacro.load_yaml('$(arg initial_positions_file)')}"/>
   <xacro:include
     filename="$(find ur_description)/urdf/ur_macro.xacro"/>
@@ -20,3 +29,65 @@
     <origin xyz="0 0 0" rpy="0 0 0"/>
   </xacro:ur_robot>
+  <ros2_control name="MujocoSystem" type="system">
+    <hardware>
+      <plugin>mujoco_ros2_control/MujocoSystemInterface</plugin>
+      <param name="mujoco_model">$(arg mujoco_model)</param>
+      <param name="headless">false</param>
+    </hardware>
+    <!-- six UR5e joints -->
+    <joint name="shoulder_pan_joint">
+      <command_interface name="position"/>
+      <state_interface name="position">
+        <param name="initial_value">
+          ${initial_positions['shoulder_pan_joint']}
+        </param>
+      </state_interface>
+      <state_interface name="velocity"/>
+    </joint>
+    <joint name="shoulder_lift_joint">
+      <command_interface name="position"/>
+      <state_interface name="position">
+        <param name="initial_value">
+          ${initial_positions['shoulder_lift_joint']}
+        </param>
+      </state_interface>
+      <state_interface name="velocity"/>
+    </joint>
+    <joint name="elbow_joint">
+      <command_interface name="position"/>
+      <state_interface name="position">
+        <param name="initial_value">
+          ${initial_positions['elbow_joint']}
+        </param>
+      </state_interface>
+      <state_interface name="velocity"/>
+    </joint>
+    <joint name="wrist_1_joint">
+      <command_interface name="position"/>
+      <state_interface name="position">
+        <param name="initial_value">
+          ${initial_positions['wrist_1_joint']}
+        </param>
+      </state_interface>
+      <state_interface name="velocity"/>
+    </joint>
+    <joint name="wrist_2_joint">
+      <command_interface name="position"/>
+      <state_interface name="position">
+        <param name="initial_value">
+          ${initial_positions['wrist_2_joint']}
+        </param>
+      </state_interface>
+      <state_interface name="velocity"/>
+    </joint>
+    <joint name="wrist_3_joint">
+      <command_interface name="position"/>
+      <state_interface name="position">
+        <param name="initial_value">
+          ${initial_positions['wrist_3_joint']}
+        </param>
+      </state_interface>
+      <state_interface name="velocity"/>
+    </joint>
+  </ros2_control>
 </robot>
