Commit message: Separate UR5e description from MuJoCo simulation

File: src/ur5e_mujoco_sim/urdf/ur5e.urdf.xacro (robot description, xacro)
@@ -13,20 +13,9 @@
     value="${xacro.load_yaml('$(arg initial_positions_file)')}"/>
   <xacro:include
-    filename="$(find ur_description)/urdf/ur_macro.xacro"/>
+    filename="$(find ur5e_description)/urdf/ur5e_macro.xacro"/>
   <link name="world"/>
-  <xacro:ur_robot
-    name="ur5e"
-    tf_prefix=""
+  <xacro:ur5e_robot
     parent="world"
-    joint_limits_parameters_file="$(find ur_description)/config/ur5e/joint_limits.yaml"
-    kinematics_parameters_file="$(find ur_description)/config/ur5e/default_kinematics.yaml"
-    physical_parameters_file="$(find ur_description)/config/ur5e/physical_parameters.yaml"
-    visual_parameters_file="$(find ur_description)/config/ur5e/visual_parameters.yaml"
-    safety_limits="false"
-    safety_pos_margin="0.15"
-    safety_k_position="20"
-    force_abs_paths="true">
-    <origin xyz="0 0 0" rpy="0 0 0"/>
-  </xacro:ur_robot>
+    tf_prefix=""/>
   <ros2_control name="MujocoSystem" type="system">
     <hardware>
